Commit message: WOrking on manipulator

File: hera_description/urdf/manip_prop.urdf.xacro (robot description, xacro)
@@ -6,6 +6,6 @@
             <origin xyz="0.00030938336056912 -9.89895665437501E-13 0.0229511892881233" rpy="0 0 0" />
             <mass value="${mass}" />
-            <inertia ixx="5.65453718592828E-05" ixy="5.00162232371705E-16"  ixz="-1.38639831470138E-06"
-                     iyy="0.000101241328443196" iyz="-3.18870100704921E-15" izz="8.47747908239031E-05" />
+            <inertia ixx="0.002" ixy="0.0"  ixz="0.0"
+                     iyy="0.02" iyz="0.0" izz="0.002"/>
         </inertial>
     </xacro:macro>
@@ -15,6 +15,6 @@
             <origin xyz="0.010403379929175 1.63335446591584E-08 0.0169657675518438" rpy="0 0 0" />
             <mass value="${mass}" />
-            <inertia ixx="2.12284942933575E-05" ixy="2.48129475489142E-12" ixz="-1.76897405605609E-06"
-                     iyy="1.25993311294143E-05" iyz="3.2054762687646E-12"  izz="2.59552674841784E-05" />
+            <inertia ixx="0.002" ixy="0.0"  ixz="0.0"
+                     iyy="0.02" iyz="0.0" izz="0.002"/>
         </inertial>
     </xacro:macro>
@@ -24,6 +24,6 @@
             <origin xyz="0.0763705857165563 0.000254475982597022 0.00808212627192917" rpy="0 0 0" />
             <mass value="${mass}" />
-            <inertia ixx="0.000193142254231562" ixy="4.37085471306953E-07"  ixz="-1.72353751616987E-05"
-                     iyy="0.000387146626280563" iyz="-1.13959846344025E-12" izz="0.000310532195206607"/>
+            <inertia ixx="0.002" ixy="0.0"  ixz="0.0"
+                     iyy="0.02" iyz="0.0" izz="0.002"/>
         </inertial>
     </xacro:macro>
@@ -33,6 +33,6 @@
             <origin xyz="0.0169657676446836 1.64819090528456E-08 -0.0104033800071373" rpy="0 0 0" />
             <mass value="${mass}" />
-            <inertia ixx="2.5955267230398E-05"  ixy="3.22328296007298E-12"  ixz="1.76897404833607E-06"
-                     iyy="1.25993310604571E-05" iyz="-2.56726778703582E-12" izz="2.12284940766909E-05"/>
+            <inertia ixx="0.002" ixy="0.0"  ixz="0.0"
+                     iyy="0.02" iyz="0.0" izz="0.002"/>
         </inertial>
     </xacro:macro>
@@ -42,6 +42,6 @@
             <origin xyz="0.0763705857419602 -0.00025447598295664 0.00808212650131321" rpy="0 0 0" />
             <mass value="${mass}" />
-            <inertia ixx="0.000193142254252889" ixy="-4.37085476272942E-07" ixz="-1.72353755052685E-05"
-                     iyy="0.000387146626356831" iyz="-1.13953084591342E-12" izz="0.000310532195285594"/>
+            <inertia ixx="0.002" ixy="0.0"  ixz="0.0"
+                     iyy="0.02" iyz="0.0" izz="0.002"/>
         </inertial>
     </xacro:macro>
@@ -51,6 +51,6 @@
             <origin xyz="0.0113429838803915 -3.46944695195361E-18 0" rpy="0 0 0" />
             <mass value="${mass}" />
-            <inertia ixx="1.95927087211338E-05" ixy="7.26329421268603E-21" ixz="-2.5410988417629E-21"
-                     iyy="7.36984687037621E-06" iyz="8.60646127431738E-21" izz="2.02402124370273E-05" />
+            <inertia ixx="0.002" ixy="0.0"  ixz="0.0"
+                     iyy="0.02" iyz="0.0" izz="0.002"/>
         </inertial>
     </xacro:macro>
@@ -61,7 +61,6 @@
                     rpy="0 0 0" />
             <mass value="${mass}" />
-            <inertia ixx="0.000146386226397184" ixy="-4.37085473836754E-07" ixz="-1.5900787088928E-13"
-                     iyy="0.000125206462596505" iyz="-1.1391259066856E-12"
-                     izz="0.000181710835049005"/>
+            <inertia ixx="0.002" ixy="0.0"  ixz="0.0"
+                     iyy="0.02" iyz="0.0" izz="0.002"/>
         </inertial>
     </xacro:macro>
@@ -72,6 +71,6 @@
                     rpy="0 0 0" />
             <mass value="${mass}" />
-            <inertia ixx="1.12762059938717E-05" ixy="2.39164603983455E-07" ixz="-1.49908527899727E-12"
-                     iyy="1.06667583466197E-05" iyz="1.51683951155461E-12" izz="3.59815370093277E-06" />
+            <inertia ixx="0.002" ixy="0.0"  ixz="0.0"
+                     iyy="0.02" iyz="0.0" izz="0.002"/>
         </inertial>
     </xacro:macro>
@@ -82,6 +81,6 @@
                     rpy="0 0 0" />
             <mass value="${mass}" />
-            <inertia ixx="2.29035041365173E-05" ixy="-1.8272694134383E-05" ixz="-1.47284953313777E-11"
-                     iyy="5.672487088308E-05" iyz="-6.47534317160686E-12" izz="5.94928785230653E-05" />
+            <inertia ixx="0.002" ixy="0.0"  ixz="0.0"
+                     iyy="0.02" iyz="0.0" izz="0.002"/>
         </inertial>
     </xacro:macro>
@@ -92,6 +91,6 @@
                     rpy="0 0 0" />
             <mass value="${mass}" />
-            <inertia ixx="2.29035009049597E-05" ixy="1.82727115379582E-05" ixz="3.07510207373307E-11"
-                     iyy="5.67249052626609E-05" iyz="-1.11321771779834E-11" izz="5.94929088813273E-05" />
+            <inertia ixx="0.002" ixy="0.0"  ixz="0.0"
+                     iyy="0.02" iyz="0.0" izz="0.002"/>
         </inertial>
     </xacro:macro>
@@ -102,6 +101,6 @@
                     rpy="0 0 0" />
             <mass value="${mass}" />
-            <inertia ixx="2.29035009049597E-05" ixy="1.82727115379582E-05" ixz="3.07510207373307E-11"
-                     iyy="5.67249052626609E-05" iyz="-1.11321771779834E-11" izz="5.94929088813273E-05" />
+            <inertia ixx="0.002" ixy="0.0"  ixz="0.0"
+                     iyy="0.02" iyz="0.0" izz="0.002"/>
         </inertial>
     </xacro:macro>
@@ -111,6 +110,6 @@
             <origin xyz="0.099437810671345 2.00188811166901E-07 0.0198713294048926" rpy="0 0 0" />
             <mass value="${mass}" />
-            <inertia ixx="0.000498685766551954" ixy="4.35797776215065E-09" ixz="-0.000221629766113691"
-                     iyy="0.00233391280566028"  iyz="5.90356892037055E-09" izz="0.00260971250229957" />
+            <inertia ixx="0.002" ixy="0.0"  ixz="0.0"
+                     iyy="0.02" iyz="0.0" izz="0.002"/>
         </inertial>
     </xacro:macro>
@@ -120,6 +119,6 @@
             <origin xyz="0.00515298283191654 -0.00667089588666656 0.110700863109422" rpy="0 0 0" />
             <mass value="${mass}" />
-            <inertia ixx="0.00019606850493542"  ixy="-8.60297419203407E-20" ixz="-4.60131708471049E-20"
-                     iyy="0.000183353038292849" iyz="-1.01509944145167E-19" izz="2.15450520465379E-05" />
+            <inertia ixx="0.002" ixy="0.0"  ixz="0.0"
+                     iyy="0.02" iyz="0.0" izz="0.002"/>
         </inertial>
     </xacro:macro>

File: hera_description/urdf/simulation/manip_transmission.xacro (robot description, xacro)
@@ -5,8 +5,8 @@
       <type>transmission_interface/SimpleTransmission</type>
       <joint name="joint_1">
-        <hardwareInterface>hardware_interface/PositionJointInterface</hardwareInterface>
+        <hardwareInterface>hardware_interface/EffortJointInterface</hardwareInterface>
       </joint>
       <actuator name="joint_1_motor">
-        <hardwareInterface>hardware_interface/PositionJointInterface</hardwareInterface>
+        <hardwareInterface>hardware_interface/EffortJointInterface</hardwareInterface>
         <mechanicalReduction>1</mechanicalReduction>
       </actuator>
@@ -15,8 +15,8 @@
       <type>transmission_interface/SimpleTransmission</type>
       <joint name="joint_2">
-        <hardwareInterface>hardware_interface/PositionJointInterface</hardwareInterface>
+        <hardwareInterface>hardware_interface/EffortJointInterface</hardwareInterface>
       </joint>
       <actuator name="joint_2_motor">
-        <hardwareInterface>hardware_interface/PositionJointInterface</hardwareInterface>
+        <hardwareInterface>hardware_interface/EffortJointInterface</hardwareInterface>
         <mechanicalReduction>1</mechanicalReduction>
       </actuator>
@@ -25,8 +25,8 @@
       <type>transmission_interface/SimpleTransmission</type>
       <joint name="joint_3">
-        <hardwareInterface>hardware_interface/PositionJointInterface</hardwareInterface>
+        <hardwareInterface>hardware_interface/EffortJointInterface</hardwareInterface>
       </joint>
       <actuator name="joint_3_motor">
-        <hardwareInterface>hardware_interface/PositionJointInterface</hardwareInterface>
+        <hardwareInterface>hardware_interface/EffortJointInterface</hardwareInterface>
         <mechanicalReduction>1</mechanicalReduction>
       </actuator>
@@ -35,8 +35,8 @@
       <type>transmission_interface/SimpleTransmission</type>
       <joint name="joint_4">
-        <hardwareInterface>hardware_interface/PositionJointInterface</hardwareInterface>
+        <hardwareInterface>hardware_interface/EffortJointInterface</hardwareInterface>
       </joint>
       <actuator name="joint_4_motor">
-        <hardwareInterface>hardware_interface/PositionJointInterface</hardwareInterface>
+        <hardwareInterface>hardware_interface/EffortJointInterface</hardwareInterface>
         <mechanicalReduction>1</mechanicalReduction>
       </actuator>
@@ -45,8 +45,8 @@
       <type>transmission_interface/SimpleTransmission</type>
       <joint name="joint_5">
-        <hardwareInterface>hardware_interface/PositionJointInterface</hardwareInterface>
+        <hardwareInterface>hardware_interface/EffortJointInterface</hardwareInterface>
       </joint>
       <actuator name="joint_5_motor">
-        <hardwareInterface>hardware_interface/PositionJointInterface</hardwareInterface>
+        <hardwareInterface>hardware_interface/EffortJointInterface</hardwareInterface>
         <mechanicalReduction>1</mechanicalReduction>
       </actuator>
@@ -55,8 +55,8 @@
       <type>transmission_interface/SimpleTransmission</type>
       <joint name="joint_6">
-        <hardwareInterface>hardware_interface/PositionJointInterface</hardwareInterface>
+        <hardwareInterface>hardware_interface/EffortJointInterface</hardwareInterface>
       </joint>
       <actuator name="joint_6_motor">
-        <hardwareInterface>hardware_interface/PositionJointInterface</hardwareInterface>
+        <hardwareInterface>hardware_interface/EffortJointInterface</hardwareInterface>
         <mechanicalReduction>1</mechanicalReduction>
       </actuator>
@@ -66,8 +66,8 @@
       <type>transmission_interface/SimpleTransmission</type>
       <joint name="finger_1_joint_1">
-        <hardwareInterface>hardware_interface/PositionJointInterface</hardwareInterface>
+        <hardwareInterface>hardware_interface/EffortJointInterface</hardwareInterface>
       </joint>
       <actuator name="finger_1_joint_1_motor">
-        <hardwareInterface>hardware_interface/PositionJointInterface</hardwareInterface>
+        <hardwareInterface>hardware_interface/EffortJointInterface</hardwareInterface>
         <mechanicalReduction>1</mechanicalReduction>
       </actuator>
@@ -76,8 +76,8 @@
       <type>transmission_interface/SimpleTransmission</type>
       <joint name="finger_1_joint_2">
-        <hardwareInterface>hardware_interface/PositionJointInterface</hardwareInterface>
+        <hardwareInterface>hardware_interface/EffortJointInterface</hardwareInterface>
       </joint>
       <actuator name="finger_1_joint_2_motor">
-        <hardwareInterface>hardware_interface/PositionJointInterface</hardwareInterface>
+        <hardwareInterface>hardware_interface/EffortJointInterface</hardwareInterface>
         <mechanicalReduction>1</mechanicalReduction>
       </actuator>
@@ -86,8 +86,8 @@
       <type>transmission_interface/SimpleTransmission</type>
       <joint name="finger_2_joint_1">
-        <hardwareInterface>hardware_interface/PositionJointInterface</hardwareInterface>
+        <hardwareInterface>hardware_interface/EffortJointInterface</hardwareInterface>
       </joint>
       <actuator name="finger_2_joint_1_motor">
-        <hardwareInterface>hardware_interface/PositionJointInterface</hardwareInterface>
+        <hardwareInterface>hardware_interface/EffortJointInterface</hardwareInterface>
         <mechanicalReduction>1</mechanicalReduction>
       </actuator>
@@ -96,8 +96,8 @@
       <type>transmission_interface/SimpleTransmission</type>
       <joint name="finger_2_joint_2">
-        <hardwareInterface>hardware_interface/PositionJointInterface</hardwareInterface>
+        <hardwareInterface>hardware_interface/EffortJointInterface</hardwareInterface>
       </joint>
       <actuator name="finger_2_joint_2_motor">
-        <hardwareInterface>hardware_interface/PositionJointInterface</hardwareInterface>
+        <hardwareInterface>hardware_interface/EffortJointInterface</hardwareInterface>
         <mechanicalReduction>1</mechanicalReduction>
       </actuator>
@@ -106,8 +106,8 @@
       <type>transmission_interface/SimpleTransmission</type>
       <joint name="finger_middle_joint_1">
-        <hardwareInterface>hardware_interface/PositionJointInterface</hardwareInterface>
+        <hardwareInterface>hardware_interface/EffortJointInterface</hardwareInterface>
       </joint>
       <actuator name="finger_middle_joint_1_motor">
-        <hardwareInterface>hardware_interface/PositionJointInterface</hardwareInterface>
+        <hardwareInterface>hardware_interface/EffortJointInterface</hardwareInterface>
         <mechanicalReduction>1</mechanicalReduction>
       </actuator>
@@ -116,8 +116,8 @@
       <type>transmission_interface/SimpleTransmission</type>
       <joint name="finger_middle_joint_2">
-        <hardwareInterface>hardware_interface/PositionJointInterface</hardwareInterface>
+        <hardwareInterface>hardware_interface/EffortJointInterface</hardwareInterface>
       </joint>
       <actuator name="finger_middle_joint_2_motor">
-        <hardwareInterface>hardware_interface/PositionJointInterface</hardwareInterface>
+        <hardwareInterface>hardware_interface/EffortJointInterface</hardwareInterface>
         <mechanicalReduction>1</mechanicalReduction>
       </actuator>
