Commit message: Changed manip's effort limits

File: hera_description/urdf/actuators/manip.urdf.xacro (robot description, xacro)
@@ -58,5 +58,6 @@
       <child link="link_1" />
       <axis xyz="0 0 1" />
-      <limit lower="-3.14" upper="3.14" effort="8" velocity="5" />
+      <limit lower="-3.14" upper="3.14" effort="0.0" velocity="1.0" />
+      <dynamics damping="10.0" friction="100.0" />
     </joint>
   </xacro:macro>
@@ -87,5 +88,6 @@
       <child link="link_2" />
       <axis xyz="0 1 0" />
-      <limit lower="-2.355" upper="3.14" effort="8" velocity="5" />
+      <limit lower="-2.355" upper="3.14" effort="0.0" velocity="1.0" />
+      <dynamics damping="10.0" friction="100.0" />
     </joint>
   </xacro:macro>
@@ -116,5 +118,6 @@
       <child link="link_3" />
       <axis xyz="1 0 0" />
-      <limit lower="-3.14" upper="3.14" effort="8" velocity="5" />
+      <limit lower="-3.14" upper="3.14" effort="0.0" velocity="1.0" />
+      <dynamics damping="10.0" friction="100.0" />
     </joint>
   </xacro:macro>
@@ -145,5 +148,6 @@
       <child link="link_4" />
       <axis xyz="0 -1 0" />
-      <limit lower="-3.14" upper="1.0078" effort="8" velocity="5" />
+      <limit lower="-3.14" upper="1.0078" effort="0.0" velocity="1.0" />
+      <dynamics damping="10.0" friction="100.0" />
     </joint>
   </xacro:macro>
@@ -174,5 +178,6 @@
       <child link="link_5" />
       <axis xyz="1 0 0" />
-      <limit lower="-3.14" upper="3.14" effort="8" velocity="5" />
+      <limit lower="-3.14" upper="3.14" effort="0.0" velocity="1.0" />
+      <dynamics damping="10.0" friction="100.0" />
     </joint>
   </xacro:macro>
@@ -203,5 +208,6 @@
       <child link="link_6" />
       <axis xyz="0 -1 0" />
-      <limit lower="-2.6232" upper="1.8262" effort="8" velocity="5" />
+      <limit lower="-2.6232" upper="1.8262" effort="0.0" velocity="1.0" />
+      <dynamics damping="10.0" friction="100.0" />
     </joint>
   </xacro:macro>
