Commit message: suporte_joint revolute and configs

File: hera_description/urdf/actuators/torso.urdf.xacro (robot description, xacro)
@@ -143,10 +143,10 @@
     </link>
     <!--suporte_joint-->
-    <joint name="suporte_joint" type="fixed">
+    <joint name="suporte_joint" type="revolute">
       <origin xyz="0.04525 0 0.0285" rpy="0 0 0" />
       <parent link="${parent}" />
       <child link="suporte_link" />
-      <axis xyz="0 0 0" />
-      <limit lower="0" upper="0" effort="0" velocity="0" />
+      <axis xyz="0 1 0" />
+      <limit lower="0.0" upper="1.57" effort="100" velocity="100" />
     </joint>
   </xacro:macro>

File: hera_description/urdf/simulation/manip_transmission.xacro (robot description, xacro)
@@ -123,4 +123,21 @@
       </actuator>
     </transmission>
+  <!--##################### SUPORT ########################-->
+    <gazebo>
+        <plugin name="gazebo_ros_control" filename="libgazebo_ros_control.so">
+        <robotNamespace>/suport</robotNamespace>
+        <robotSimType>gazebo_ros_control/DefaultRobotHWSim</robotSimType>
+        </plugin>
+    </gazebo>
+    <transmission name="trans_suport">
+      <type>transmission_interface/SimpleTransmission</type>
+      <joint name="suporte_joint">
+        <hardwareInterface>hardware_interface/EffortJointInterface</hardwareInterface>
+      </joint>
+      <actuator name="suporte_joint_motor">
+        <hardwareInterface>hardware_interface/EffortJointInterface</hardwareInterface>
+        <mechanicalReduction>1</mechanicalReduction>
+      </actuator>
+    </transmission>
   </xacro:macro>
 </robot>

Commit message: Added kinect controller

File: hera_description/urdf/actuators/torso.urdf.xacro (robot description, xacro)
@@ -102,8 +102,11 @@
     </joint>
     <!-- should be revolute -->
-    <joint name="joint_${name}_to_${name}_sensor_plat" type="fixed">
+    <joint name="joint_${name}_to_${name}_sensor_plat" type="revolute">
       <origin xyz="0.09 0 0.46" rpy="0 0 0"/> <!-- rpy="0 0 0" -->
       <parent link="${name}"/>
       <child link="${name}_sensor_plat"/>
+      <axis xyz="0 1 0"/> -->
+      <limit effort="${torso_sensor_plat_effort}" velocity="${torso_sensor_plat_velocity}"
+        lower="0.0" upper="1.57"/>
     </joint>
   </xacro:macro>

File: hera_description/urdf/gazebo/manipulator.gazebo.xacro (robot description, xacro)
@@ -100,4 +100,12 @@
       </joint>
     </transmission>
+    <transmission name="kinect_trans">
+      <type>transmission_interface/SimpleTransmission</type>
+      <actuator name="torso_to_torso_sensor_plat_motor" >
+      </actuator>
+      <joint name="joint_torso_to_torso_sensor_plat">
+        <hardwareInterface>hardware_interface/PositionJointInterface</hardwareInterface>
+      </joint>
+    </transmission>
 <!--##################### ROS CONTROL ########################-->
     <gazebo>
@@ -108,11 +116,11 @@
     </gazebo>
 <!--##################### GRASP FIX ########################-->
-    <!-- <gazebo>
+    <gazebo>
         <plugin name="gazebo_grasp_fix" filename="libgazebo_grasp_fix.so">
              <arm>
-                <arm_name>hera_arm</arm_name>
-                <palm_link> wrist_lift_link  </palm_link>
-                <gripper_link> gripper_left_link </gripper_link>
-                <gripper_link> gripper_right_link </gripper_link>
+                <arm_name>arm</arm_name>
+                <palm_link> wrist_lift_link</palm_link>
+                <gripper_link> gripper_left_finger_link</gripper_link>
+                <gripper_link> gripper_right_finger_link</gripper_link>
              </arm>
             <forces_angle_tolerance>100</forces_angle_tolerance>
@@ -121,8 +129,8 @@
             <max_grip_count>8</max_grip_count>
             <release_tolerance>0.005</release_tolerance>
-            <disable_collisions_on_attach>true</disable_collisions_on_attach>
+            <disable_collisions_on_attach>false</disable_collisions_on_attach>
             <contact_topic>__default_topic__</contact_topic>
         </plugin>
-      </gazebo> -->
+      </gazebo>
   </xacro:macro>
 </robot>
