Commit message: Fixed support names

File: hera_description/robots/hera_full.urdf.xacro (robot description, xacro)
@@ -70,5 +70,5 @@
   </xacro:kinect_one>
   <!--torso suporte-->
-  <xacro:create_suporte_link
+  <xacro:create_support_link
     parent="torso"/>
   <!--torso encosto-->

File: hera_description/urdf/actuators/manip.urdf.xacro (robot description, xacro)
@@ -26,5 +26,5 @@
     <joint name="base_joint" type="fixed">
       <origin xyz="0.27075 0 0.0295" rpy="0 0 0" />
-      <parent link="suporte_link" />
+      <parent link="support_link" />
       <child link="base_link" />
       <axis xyz="0 0 0" />

File: hera_description/urdf/actuators/torso.urdf.xacro (robot description, xacro)
@@ -122,11 +122,11 @@
     </transmission>
   </xacro:macro>
-  <!--suporte_link-->
-  <xacro:macro name="create_suporte_link" params="parent">
-    <link name="suporte_link">
+  <!--support_link-->
+  <xacro:macro name="create_support_link" params="parent">
+    <link name="support_link">
       <visual>
         <origin xyz="0 0 0" rpy="0 0 0" />
         <geometry>
-          <mesh filename="package://hera_description/meshes/manip_meshes/suporte_link.STL"/>
+          <mesh filename="package://hera_description/meshes/manip_meshes/support_link.STL"/>
         </geometry>
         <material name="grey">
@@ -137,14 +137,14 @@
         <origin xyz="0 0 0" rpy="0 0 0" />
         <geometry>
-          <mesh filename="package://hera_description/meshes/manip_meshes/suporte_link.STL"/>
+          <mesh filename="package://hera_description/meshes/manip_meshes/support_link.STL"/>
         </geometry>
       </collision>
-      <xacro:inertial_suporte_link mass="0.659217140679788"/>
+      <xacro:inertial_support_link mass="0.659217140679788"/>
     </link>
-    <!--suporte_joint-->
-    <joint name="suporte_joint" type="revolute">
+    <!--support_joint-->
+    <joint name="support_joint" type="revolute">
       <origin xyz="0.04525 0 0.0285" rpy="0 0 0" />
       <parent link="${parent}" />
-      <child link="suporte_link" />
+      <child link="support_link" />
       <axis xyz="0 1 0" />
       <limit lower="0.0" upper="1.57" effort="100" velocity="100" />

File: hera_description/urdf/manip_prop.urdf.xacro (robot description, xacro)
@@ -106,6 +106,6 @@
         </inertial>
     </xacro:macro>
-<!--inertial_suporte_link-->
-    <xacro:macro name="inertial_suporte_link" params="mass">
+<!--inertial_support_link-->
+    <xacro:macro name="inertial_support_link" params="mass">
         <inertial>
             <origin xyz="0.099437810671345 2.00188811166901E-07 0.0198713294048926" rpy="0 0 0" />

File: hera_description/urdf/simulation/manip_transmission.xacro (robot description, xacro)
@@ -123,17 +123,17 @@
       </actuator>
     </transmission>
-  <!--##################### SUPORT ########################-->
+  <!--##################### support ########################-->
     <gazebo>
         <plugin name="gazebo_ros_control" filename="libgazebo_ros_control.so">
-        <robotNamespace>/suport</robotNamespace>
+        <robotNamespace>/support</robotNamespace>
         <robotSimType>gazebo_ros_control/DefaultRobotHWSim</robotSimType>
         </plugin>
     </gazebo>
-    <transmission name="trans_suport">
+    <transmission name="trans_support">
       <type>transmission_interface/SimpleTransmission</type>
-      <joint name="suporte_joint">
+      <joint name="support_joint">
         <hardwareInterface>hardware_interface/EffortJointInterface</hardwareInterface>
       </joint>
-      <actuator name="suporte_joint_motor">
+      <actuator name="support_joint_motor">
         <hardwareInterface>hardware_interface/EffortJointInterface</hardwareInterface>
         <mechanicalReduction>1</mechanicalReduction>

Commit message: new gripper on urdf

File: hera_description/robots/hera_full.urdf.xacro (robot description, xacro)
@@ -106,5 +106,5 @@
   <xacro:gazebo_manip/>
   <!-- gripper_contact_sensors -->
-  <xacro:gripper_contact_sensors/>
+  <!-- <xacro:gripper_contact_sensors/> -->
 <!-- ####################################################################### -->
 <!-- ####################### gazebo sensors #################################-->

File: hera_description/urdf/actuators/manip.urdf.xacro (robot description, xacro)
@@ -3,5 +3,6 @@
 <xacro:include filename="$(find hera_description)/urdf/manip_prop.urdf.xacro"/>
 <xacro:include filename="$(find hera_description)/urdf/simulation/manip_transmission.xacro"/>
-<xacro:include filename="$(find hera_description)/urdf/actuators/gripper/robotiq-3f-gripper_articulated_macro.xacro"/>
+<!-- <xacro:include filename="$(find hera_description)/urdf/actuators/gripper/robotiq-3f-gripper_articulated_macro.xacro"/> -->
+<xacro:include filename="$(find pal_gripper_description)/urdf/gripper.urdf.xacro" />
 <!--base_link-->
   <xacro:macro name="create_base_link">
@@ -222,5 +223,8 @@
     <xacro:create_link_6/>
     <!-- Gripper -->
-    <xacro:robotiq-3f-gripper_articulated prefix=""/>
+    <!-- <xacro:robotiq-3f-gripper_articulated prefix=""/> -->
+    <xacro:pal_gripper parent="link_6" name="gripper">
+      <origin xyz="0.06 0 0" rpy="0 -1.57 0" />
+    </xacro:pal_gripper>
     <!--Transmission-->
     <xacro:manip_transmission/>

Commit message: Rework on hera_description

File: hera_description/robots/hera_full.urdf.xacro (robot description, xacro)
@@ -15,5 +15,5 @@
   <xacro:include filename="$(find hera_description)/urdf/actuators/torso.urdf.xacro" />
   <xacro:include filename="$(find hera_description)/urdf/actuators/head.urdf.xacro" />
-  <xacro:include filename="$(find hera_description)/urdf/actuators/manip.urdf.xacro" />
+  <xacro:include filename="$(find hera_description)/urdf/actuators/manipulator/manip.urdf.xacro" />
   <!-- sensors -->
   <xacro:include filename="$(find hera_description)/urdf/sensors/hokuyo_utm.urdf.xacro"/>
@@ -21,14 +21,12 @@
   <xacro:include filename="$(find hera_description)/urdf/sensors/asus_xtion.urdf.xacro"/>
   <xacro:include filename="$(find hera_description)/urdf/sensors/kinect_one.urdf.xacro"/>
-  <xacro:include filename="$(find hera_description)/urdf/sensors/gripper_contact_sensors.urdf.xacro"/>
   <!-- simulation -->
-  <xacro:include filename="$(find hera_description)/urdf/simulation/colors.gazebo.xacro" />
-  <xacro:include filename="$(find hera_description)/urdf/simulation/control.gazebo.xacro" />
-  <xacro:include filename="$(find hera_description)/urdf/simulation/base.gazebo.xacro"/>
-  <xacro:include filename="$(find hera_description)/urdf/simulation/hokuyo_utm.gazebo.xacro" />
-  <xacro:include filename="$(find hera_description)/urdf/simulation/hokuyo_urg.gazebo.xacro" />
-  <xacro:include filename="$(find hera_description)/urdf/simulation/asus_xtion.gazebo.xacro" />
-  <xacro:include filename="$(find hera_description)/urdf/simulation/kinect_one.gazebo.xacro" />
-  <xacro:include filename="$(find hera_description)/urdf/simulation/manip.gazebo.xacro" />
+  <xacro:include filename="$(find hera_description)/urdf/gazebo/colors.gazebo.xacro" />
+  <xacro:include filename="$(find hera_description)/urdf/gazebo/base.gazebo.xacro"/>
+  <xacro:include filename="$(find hera_description)/urdf/gazebo/hokuyo_utm.gazebo.xacro" />
+  <xacro:include filename="$(find hera_description)/urdf/gazebo/hokuyo_urg.gazebo.xacro" />
+  <xacro:include filename="$(find hera_description)/urdf/gazebo/asus_xtion.gazebo.xacro" />
+  <xacro:include filename="$(find hera_description)/urdf/gazebo/kinect_one.gazebo.xacro" />
+  <xacro:include filename="$(find hera_description)/urdf/gazebo/manipulator.gazebo.xacro" />
 <!-- ####################################################################### -->
 <!-- ######################## robot parts ################################## -->
@@ -70,11 +68,11 @@
   </xacro:kinect_one>
   <!--torso suporte-->
-  <xacro:create_support_link
+  <xacro:create_manip_support_link
     parent="torso"/>
-  <!--torso encosto-->
-  <xacro:create_encosto_link
+  <!--torso backrest-->
+  <xacro:create_backrest_link
     parent="torso"/>
   <!-- manip -->
-  <xacro:manip/>
+  <xacro:manipulator/>
 <!-- ####################################################################### -->
 <!-- ####################### gazebo extensions ##############################-->
@@ -103,51 +101,4 @@
     reference="kinect_one"
     update_rate="30"/>
-  <!-- manip_plugin -->
-  <xacro:gazebo_manip/>
-  <!-- gripper_contact_sensors -->
-  <!-- <xacro:gripper_contact_sensors/> -->
-<!-- ####################################################################### -->
-<!-- ####################### gazebo sensors #################################-->
-<!-- ####################################################################### -->
-  <!-- <gazebo reference="link_6">
-    <turnGravityOff>true</turnGravityOff>
-    <selfCollide>false</selfCollide>
-    <sensor type="contact" name="palm_contactsensor_sensor">
-      <update_rate>100.0</update_rate>
-      <contact>
-        <collision>link_6_fixed_joint_lump__palm_collision_1</collision>
-      </contact>
-      <plugin name="palm_plugin" filename="libgazebo_ros_bumper.so">
-        <alwaysOn>true</alwaysOn>
-        <frameName>link_6</frameName>
-        <updateRate>100.0</updateRate>
-        <bumperTopicName>link_6_bumper</bumperTopicName>
-      </plugin>
-    </sensor>
-    <mu1 value="500.0" />
-    <mu2 value="500.0" />
-    <kp  value="10000000.0" />
-    <kd  value="1.0" />
-  </gazebo> -->
-  <!-- FINGER 1 LINK 3 SENSOR
-  <gazebo reference="finger_1_link_3">
-    <turnGravityOff>true</turnGravityOff>
-    <selfCollide>false</selfCollide>
-    <sensor type="contact" name="finger_1_link_3_contactsensor_sensor">
-      <alwaysOn>true</alwaysOn>
-      <update_rate>100.0</update_rate>
-      <contact>
-        <collision>finger_1_link_2_fixed_joint_lump__finger_1_link_3_collision_1</collision>
-      </contact>
-      <plugin name="finger_1_link_3_plugin" filename="libgazebo_ros_bumper.so">
-        <bumperTopicName>finger_1_link_3_bumper</bumperTopicName>
-        <frameName>finger_1_link_3</frameName>
-      </plugin>
-    </sensor>
-    <mu1 value="500.0" />
-    <mu2 value="500.0" />
-    <kp  value="10000000.0" />
-    <kd  value="1.0" />
-    <provideFeedback value="true"/>
-  </gazebo> -->
+  <xacro:manip_transmission/>
 </robot>

File: hera_description/urdf/actuators/base.urdf.xacro (robot description, xacro)
@@ -4,5 +4,5 @@
        xmlns:interface="http://playerstage.sourceforge.net/gazebo/xmlschema/#interface"
        xmlns:xacro="http://ros.org/wiki/xacro">
-  <xacro:property name="base_mass"      value="100.0"/>
+  <xacro:property name="base_mass"      value="99.9"/>
   <xacro:property name="base_size_x"    value="0.50"/>
   <xacro:property name="base_size_y"    value="0.30"/>

File: hera_description/urdf/actuators/head.urdf.xacro (robot description, xacro)
@@ -60,14 +60,4 @@
       <limit effort="${head_effort}" velocity="${head_velocity}" lower="-${M_PI/2}" upper="${M_PI/2}"/>
     </joint>
-    <!-- <transmission name="tran_${name}">
-      <type>transmission_interface/SimpleTransmission</type>
-      <joint name="joint_${parent}_to_${name}">
-        <hardwareInterface>hardware_interface/EffortJointInterface</hardwareInterface>
-      </joint>
-      <actuator name="motor_${name}">
-        <hardwareInterface>hardware_interface/EffortJointInterface</hardwareInterface>
-        <mechanicalReduction>1</mechanicalReduction>
-      </actuator>
-    </transmission> -->
   </xacro:macro>
 </robot>

File: hera_description/urdf/actuators/torso.urdf.xacro (robot description, xacro)
@@ -20,5 +20,5 @@
   <xacro:property name="pole_size_y"       value="0.06"/>
   <xacro:property name="pole_size_z"       value="1.00"/>
-  <xacro:property name="sensor_plat_mass"             value="1.0"/>
+  <xacro:property name="sensor_plat_mass"             value="0.01"/>
   <xacro:property name="sensor_plat_size_x"           value="0.10"/>
   <xacro:property name="sensor_plat_size_y"           value="0.12"/>
@@ -102,31 +102,17 @@
     </joint>
     <!-- should be revolute -->
-    <joint name="joint_${name}_to_${name}_sensor_plat" type="revolute">
+    <joint name="joint_${name}_to_${name}_sensor_plat" type="fixed">
       <origin xyz="0.09 0 0.46" rpy="0 0 0"/> <!-- rpy="0 0 0" -->
       <parent link="${name}"/>
       <child link="${name}_sensor_plat"/>
-      <axis xyz="0 1 0"/> -->
-      <limit effort="${torso_sensor_plat_effort}" velocity="${torso_sensor_plat_velocity}"
-        lower="0.0" upper="1.57"/>
     </joint>
-    <!-- Transmission to Gazebo Plugin -->
-    <transmission name="trans_kinect">
-      <type>transmission_interface/SimpleTransmission</type>
-      <joint name="joint_torso_to_torso_sensor_plat">
-        <hardwareInterface>hardware_interface/EffortJointInterface</hardwareInterface>
-      </joint>
-      <actuator name="kinect_motor">
-        <hardwareInterface>hardware_interface/EffortJointInterface</hardwareInterface>
-        <mechanicalReduction>1</mechanicalReduction>
-      </actuator>
-    </transmission>
   </xacro:macro>
-  <!--support_link-->
-  <xacro:macro name="create_support_link" params="parent">
-    <link name="support_link">
+  <!--manip_support_link-->
+  <xacro:macro name="create_manip_support_link" params="parent">
+    <link name="manip_support_link">
       <visual>
         <origin xyz="0 0 0" rpy="0 0 0" />
         <geometry>
-          <mesh filename="package://hera_description/meshes/manip_meshes/support_link.STL"/>
+          <mesh filename="package://hera_description/meshes/manip_meshes/manip_support.STL"/>
         </geometry>
         <material name="grey">
@@ -137,25 +123,25 @@
         <origin xyz="0 0 0" rpy="0 0 0" />
         <geometry>
-          <mesh filename="package://hera_description/meshes/manip_meshes/support_link.STL"/>
+          <mesh filename="package://hera_description/meshes/manip_meshes/manip_support.STL"/>
         </geometry>
       </collision>
-      <xacro:inertial_support_link mass="0.659217140679788"/>
+      <xacro:inertial_manip_support_link mass="0.659217140679788"/>
     </link>
-    <!--support_joint-->
-    <joint name="support_joint" type="revolute">
+    <!--manip_support_joint-->
+    <joint name="manip_support_joint" type="fixed">
       <origin xyz="0.04525 0 0.0285" rpy="0 0 0" />
       <parent link="${parent}" />
-      <child link="support_link" />
-      <axis xyz="0 1 0" />
-      <limit lower="0.0" upper="1.57" effort="100" velocity="100" />
+      <child link="manip_support_link" />
+      <axis xyz="0 0 0" />
+      <limit lower="0" upper="0" effort="0" velocity="0" />
     </joint>
   </xacro:macro>
-  <!--encosto_link-->
-  <xacro:macro name="create_encosto_link" params="parent">
-    <link name="encosto_link">
+  <!--backrest_link-->
+  <xacro:macro name="create_backrest_link" params="parent">
+    <link name="backrest_link">
       <visual>
         <origin xyz="0 0 0" rpy="0 0 0" />
         <geometry>
-          <mesh filename="package://hera_description/meshes/manip_meshes/encosto_link.STL"/>
+          <mesh filename="package://hera_description/meshes/manip_meshes/backrest.STL"/>
         </geometry>
         <material name="grey">
@@ -166,14 +152,14 @@
         <origin xyz="0 0 0" rpy="0 0 0" />
         <geometry>
-          <mesh filename="package://hera_description/meshes/manip_meshes/encosto_link.STL"/>
+          <mesh filename="package://hera_description/meshes/manip_meshes/backrest.STL"/>
         </geometry>
       </collision>
-      <xacro:inertial_base_link mass="0.0709912944888601"/>
+      <xacro:inertial_backrest_link mass="0.0709912944888601"/>
     </link>
-    <!--encosto_joint-->
-    <joint name="encosto_joint" type="fixed">
+    <!--backrest_joint-->
+    <joint name="backrest_joint" type="fixed">
       <origin xyz="0.028 0.0066709 0.053" rpy="0 0 0" />
       <parent link="${parent}" />
-      <child link="encosto_link" />
+      <child link="backrest_link" />
       <axis xyz="0 0 0" />
       <limit effort="0" velocity="0" />

File: hera_description/urdf/gazebo/asus_xtion.gazebo.xacro (robot description, xacro)
@@ -11,6 +11,6 @@
             <image>
               <format>R8G8B8</format>
-              <width>${640/20}</width>
-              <height>${480/20}</height>
+              <width>${640}</width>
+              <height>${480}</height>
             </image>
             <clip>

File: hera_description/urdf/gazebo/kinect_one.gazebo.xacro (robot description, xacro)
@@ -10,6 +10,6 @@
                 <image>
                   <format>R8G8B8</format>
-                  <width>${1280}</width>
-                  <height>${720}</height>
+                  <width>${640}</width>
+                  <height>${480}</height>
                 </image>
                 <clip>
@@ -42,10 +42,4 @@
           </sensor>
         </gazebo>
-        <gazebo>
-            <plugin name="gazebo_ros_control" filename="libgazebo_ros_control.so">
-            <robotNamespace>/kinect</robotNamespace>
-            <robotSimType>gazebo_ros_control/DefaultRobotHWSim</robotSimType>
-            </plugin>
-        </gazebo>
     </xacro:macro>
   </robot>
