Commit message: Changed limits and added mimic joint plugin

File: hera_description/urdf/actuators/manipulator/simulation_gripper/gripper.urdf.xacro (robot description, xacro)
@@ -82,11 +82,11 @@
     <child link="${name}_right_finger_link" />
     <axis xyz="1 0 0" />
-    <limit effort="16" lower="0.0" upper="0.055" velocity="0.05" />
-    <calibration rising="0.0" />
-    <dynamics damping="80" />
-    <safety_controller k_position="20"
+    <limit effort="10.0" lower="0.0" upper="0.055" velocity="1.0" />
+    <!-- <calibration rising="0.0" /> -->
+    <dynamics friction="1" damping="1" />
+    <!-- <safety_controller k_position="20"
                        k_velocity="20"
                        soft_lower_limit="${0.0 + gripper_eps}"
-                       soft_upper_limit="${0.055 - gripper_eps}" />
+                       soft_upper_limit="${0.055 - gripper_eps}" /> -->
   </joint>
   <link name="${name}_left_finger_link">
@@ -120,11 +120,12 @@
     <child link="${name}_left_finger_link" />
     <axis xyz="-1 0 0" />
-    <limit effort="16" lower="0" upper="0.055" velocity="0.05" />
-    <calibration rising="0.0" />
-    <dynamics damping="80" />
-    <safety_controller k_position="20"
+    <limit effort="10.0" lower="0" upper="0.055" velocity="1" />
+    <!-- <calibration rising="0.0" /> -->
+    <dynamics damping="1" friction="1" />
+    <!-- <safety_controller k_position="20"
                        k_velocity="20"
                        soft_lower_limit="${0.0 + gripper_eps}"
-                       soft_upper_limit="${0.055 - gripper_eps}" />
+                       soft_upper_limit="${0.055 - gripper_eps}" /> -->
+    <mimic joint="gripper_left_finger_joint" multiplier="1.0" offset="0" />
   </joint>
   <!-- Grasping frame -->

File: hera_description/urdf/gazebo/manipulator.gazebo.xacro (robot description, xacro)
@@ -89,5 +89,5 @@
       </actuator>
       <joint name="gripper_left_finger_joint">
-        <hardwareInterface>hardware_interface/PositionJointInterface</hardwareInterface>
+        <hardwareInterface>hardware_interface/EffortJointInterface</hardwareInterface>
       </joint>
     </transmission>
@@ -97,5 +97,5 @@
       </actuator>
       <joint name="gripper_right_finger_joint">
-        <hardwareInterface>hardware_interface/PositionJointInterface</hardwareInterface>
+        <hardwareInterface>hardware_interface/EffortJointInterface</hardwareInterface>
       </joint>
     </transmission>
@@ -116,4 +116,25 @@
         </plugin>
     </gazebo>
+    <xacro:macro name="mimic_joint_plugin_gazebo" params="parent_joint mimic_joint has_pid:=false multiplier:=1.0 offset:=0 sensitiveness:=0.0 max_effort:=200.0 robot_namespace:=''">
+      <gazebo>
+          <plugin name="${mimic_joint}_mimic_joint_plugin" filename="libroboticsgroup_gazebo_mimic_joint_plugin.so">
+              <joint>${parent_joint}</joint>
+              <mimicJoint>${mimic_joint}</mimicJoint>
+              <xacro:if value="${has_pid}">
+              <hasPID />
+              </xacro:if>
+              <multiplier>${multiplier}</multiplier>
+              <offset>${offset}</offset>
+              <sensitiveness>${sensitiveness}</sensitiveness>
+              <maxEffort>${max_effort}</maxEffort>
+              <xacro:unless value="${robot_namespace == ''}">
+                  <robotNamespace>($robot_namespace)</robotNamespace>
+              </xacro:unless>
+          </plugin>
+      </gazebo>
+    </xacro:macro>
+    <xacro:mimic_joint_plugin_gazebo parent_joint="gripper_left_finger_joint"
+      mimic_joint="gripper_right_finger_joint" has_pid="false" multiplier="1.0"
+      max_effort="200.0" />
 <!--##################### GRASP FIX ########################-->
     <gazebo>
