Commit message: Rotated wrist lift joint

File: hera_description/urdf/actuators/manipulator/manip.urdf.xacro (robot description, xacro)
@@ -197,5 +197,5 @@
     <!--joint_6: wrist_lift_joint-->
     <joint name="wrist_lift_joint" type="revolute">
-      <origin xyz="0.03885 0 0" rpy="0 -0.3927 0" />
+      <origin xyz="0.03885 0 0" rpy="0 1.57 0" />
       <parent link="wrist_pan_link" />
       <child link="wrist_lift_link" />

Commit message: Added Pal Gripper to simulated robot

File: hera_description/urdf/actuators/manipulator/manip.urdf.xacro (robot description, xacro)
@@ -2,4 +2,5 @@
 <robot xmlns:xacro="http://www.ros.org/wiki/xacro" name="hera_description">
 <xacro:include filename="$(find hera_description)/urdf/actuators/manipulator/manip_prop.urdf.xacro"/>
+<xacro:include filename="$(find hera_description)/urdf/actuators/manipulator/simulation_gripper/gripper.urdf.xacro" />
 <!--manip_base_link-->
   <xacro:macro name="create_manip_base_link">
@@ -334,11 +335,15 @@
     <xacro:create_wrist_lift_link/>
     <!--gripper_left_link-->
-    <xacro:create_gripper_left_link/>
+    <!-- <xacro:create_gripper_left_link/> -->
     <!--gripper_left_end_link-->
-    <xacro:create_gripper_left_end_link/>
+    <!-- <xacro:create_gripper_left_end_link/> -->
     <!--gripper_right_link-->
-    <xacro:create_gripper_right_link/>
+    <!-- <xacro:create_gripper_right_link/> -->
     <!--gripper_right_end_link-->
-    <xacro:create_gripper_right_end_link/>
+    <!-- <xacro:create_gripper_right_end_link/> -->
+    <!-- simulation_gripper -->
+    <xacro:pal_gripper parent="wrist_lift_link" name="gripper">
+      <origin xyz="0.055 0 0" rpy="0 -1.57 0" />
+    </xacro:pal_gripper>
   </xacro:macro>
 </robot>

File: hera_description/urdf/gazebo/manipulator.gazebo.xacro (robot description, xacro)
@@ -63,5 +63,5 @@
     </transmission>
 <!--##################### GRIPPER ########################-->
-    <transmission name="trans_7">
+    <!-- <transmission name="trans_7">
       <type>transmission_interface/SimpleTransmission</type>
       <joint name="gripper_left_joint">
@@ -82,4 +82,21 @@
         <mechanicalReduction>1</mechanicalReduction>
       </actuator>
+    </transmission> -->
+<!--##################### SIMULATION GRIPPER ########################-->
+    <transmission name="gripper_left_finger_trans">
+      <type>transmission_interface/SimpleTransmission</type>
+      <actuator name="gripper_left_finger_trans_motor" >
+      </actuator>
+      <joint name="gripper_left_finger_joint">
+        <hardwareInterface>hardware_interface/PositionJointInterface</hardwareInterface>
+      </joint>
+    </transmission>
+    <transmission name="gripper_right_finger_trans">
+      <type>transmission_interface/SimpleTransmission</type>
+      <actuator name="gripper_right_finger_motor" >
+      </actuator>
+      <joint name="gripper_right_finger_joint">
+        <hardwareInterface>hardware_interface/PositionJointInterface</hardwareInterface>
+      </joint>
     </transmission>
 <!--##################### ROS CONTROL ########################-->

Commit message: Added a motor on support joint

File: hera_description/urdf/actuators/manipulator/manip.urdf.xacro (robot description, xacro)
@@ -202,5 +202,5 @@
       <child link="wrist_lift_link" />
       <axis xyz="0 -1 0" />
-      <limit lower="-2.6232" upper="1.8262" effort="0" velocity="5" />
+      <limit lower="-0.4" upper="3.1415" effort="0" velocity="5" />
     </joint>
   </xacro:macro>

File: hera_description/urdf/actuators/manipulator/simulation_gripper/gripper.urdf.xacro (robot description, xacro)
@@ -120,5 +120,5 @@
     <child link="${name}_left_finger_link" />
     <axis xyz="-1 0 0" />
-    <limit effort="10.0" lower="0" upper="0.055" velocity="1" />
+    <limit effort="10.0" lower="0" upper="0.075" velocity="1" />
     <!-- <calibration rising="0.0" /> -->
     <dynamics damping="1" friction="1" />

File: hera_description/urdf/actuators/torso.urdf.xacro (robot description, xacro)
@@ -132,10 +132,10 @@
     </link>
     <!--manip_support_joint-->
-    <joint name="manip_support_joint" type="fixed">
+    <joint name="manip_support_joint" type="revolute">
       <origin xyz="0.04525 0 0.0285" rpy="0 0 0" />
       <parent link="${parent}" />
       <child link="manip_support_link" />
-      <axis xyz="0 0 0" />
-      <limit lower="0" upper="0" effort="0" velocity="0" />
+      <axis xyz="0 1 0" />
+      <limit lower="-0.5" upper="0.9" effort="0" velocity="5" />
     </joint>
   </xacro:macro>

File: hera_description/urdf/gazebo/manipulator.gazebo.xacro (robot description, xacro)
@@ -58,4 +58,14 @@
       </joint>
       <actuator name="wrist_lift_motor">
+        <hardwareInterface>hardware_interface/PositionJointInterface</hardwareInterface>
+        <mechanicalReduction>1</mechanicalReduction>
+      </actuator>
+    </transmission>
+    <transmission name="trans_7">
+      <type>transmission_interface/SimpleTransmission</type>
+      <joint name="manip_support_joint">
+        <hardwareInterface>hardware_interface/PositionJointInterface</hardwareInterface>
+      </joint>
+      <actuator name="manip_support_motor">
         <hardwareInterface>hardware_interface/PositionJointInterface</hardwareInterface>
         <mechanicalReduction>1</mechanicalReduction>
